File: PUTM_EV_TSAC_ELECTRICAL_HARNESS_2024.kicad_sch (KiCad schematic)
At the start: 45 parts, among them J1 M80-5101422, J10 M80-5100622, J12 Conn_01x06, J13 Conn_01x06, J14 M80-4800442, J15 M80-4800442, J16 M80-5100442, J17 M80-5100442, J18 M80-4800442, J19 M80-5100442, J2 M80-4801442, J20 M80-4800442, J21 M80-4800442, J22 M80-5100442, J23 M300-MV10345M1, J24 M300-225039F2, J25 M80-5100442, J26 M80-4800442, J27 Conn_01x10, J28 Conn_01x10, J29 CABLE, J3 M300-MV10345M1, J30 CABLE, J31 CABLE, J32 EYE_CONN, J33 M80-4800842, J34 M80-5100842, J35 M80-4800842, J36 Conn_01x02, J37 Conn_01x02, J38 EYE_CONN, J39 Conn_01x02, J4 M300-MV10345M1, J40 Conn_01x02, J41 M80-4800842, J42 Conn_01x37, J43 Conn_01x37, J44 TYCO 1473672-1, J45 TYCO 1473672-1, J46 M80-4803442, J5 M300-225039F2, J6 M300-225039F2, J7 M300-MV30645M1, J8 M80-5103422, J9 M80-5100442

Commit message: senpuku
Parts:
- added J11: WIRE, symbol Connector:Conn_01x02_Pin
- J32, J38: symbol Connector:Conn_01x03_Socket -> Connector:Conn_01x04_Socket
Connections:
- new net VOLTAGE_INDICATOR+: J11.2 (Pin_2), J38.4 (Pin_4)
- new net VOLTAGE_INDICATOR-: J11.1 (Pin_1), J32.4 (Pin_4)

Commit message: sync
Parts:
- removed J1: M80-5101422, symbol Connector_Generic:Conn_01x14
- removed J10: M80-5100622, symbol Connector_Generic:Conn_01x06
- removed J11: WIRE, symbol Connector:Conn_01x02_Pin
- removed J12, J13: Conn_01x06, symbol Connector_Generic:Conn_01x06
- removed J14, J15, J18, J20, J21, J26: M80-4800442, symbol Connector_Generic:Conn_01x04
- removed J16, J17, J19, J22, J25, J9: M80-5100442, symbol Connector_Generic:Conn_01x04
- removed J2: M80-4801442, symbol Connector_Generic:Conn_01x14
- removed J23, J3, J4: M300-MV10345M1, symbol Connector_Generic:Conn_01x03
- removed J24, J5, J6: M300-225039F2, symbol Connector_Generic:Conn_01x03
- removed J32, J38: EYE_CONN, symbol Connector:Conn_01x04_Socket
- removed J36, J37, J39, J40: Conn_01x02, symbol Connector_Generic:Conn_01x02
- removed J44, J45: TYCO 1473672-1, symbol Connector_Generic:Conn_01x04
- removed J46: M80-4803442, symbol Connector_Generic:Conn_01x34
- removed J7: M300-MV30645M1, symbol Connector_Generic:Conn_01x06
- removed J8: M80-5103422, symbol Connector_Generic:Conn_01x34
- added J1: M80-5102042, symbol Connector_Generic:Conn_01x20
- added J2: M80-4852042, symbol Connector_Generic:Conn_01x20
- added J3: M80-5100642, symbol Connector_Generic:Conn_01x08
- added J4: Idk man, symbol Connector_Generic:Conn_01x04
Connections:
- net 24V_IN1: no longer J28.5 (Pin_5), J42.25 (Pin_25)
- net 24V_IN2: no longer J33.1 (Pin_1), J42.27 (Pin_27)
- net AMS_CANFD1+: no longer J42.36 (Pin_36)
- net AMS_CANFD1-: no longer J42.37 (Pin_37)
- net AMS_CANFD2+: no longer J42.13 (Pin_13)
- net AMS_CANFD2-: no longer J42.14 (Pin_14)
- net AMS_CHARGER_SENS: no longer J42.17 (Pin_17)
- net AMS_EXT_RESET: no longer J42.15 (Pin_15)
- net AMS_EX_D+: no longer J42.19 (Pin_19)
- net AMS_EX_D-: no longer J42.18 (Pin_18)
- net AMS_EX_VBUS: no longer J42.12 (Pin_12)
- net AMS_USB_GND: no longer J42.28 (Pin_28)
- net GND_IN1: no longer J28.4 (Pin_4), J42.22 (Pin_22)
- net GND_IN2: no longer J33.2 (Pin_2), J33.4 (Pin_4), J42.23 (Pin_23)
- net IMD_DASH_LED: no longer J42.29 (Pin_29)
- net TSAC_SDC_IN: no longer J42.33 (Pin_33)
- net TSAL_AIR_M: no longer J28.3 (Pin_3), J42.20 (Pin_20)
- net TSAL_AIR_P: no longer J28.9 (Pin_9), J42.24 (Pin_24)
- net TSAL_AIR_PRE: no longer J28.8 (Pin_8), J42.30 (Pin_30)
- net TSAL_HV_ON: no longer J28.2 (Pin_2), J42.21 (Pin_21)
- net GND_1: now reaches J42.10 (Pin_10)
- net GND_1: now also J2.20 (Pin_20)
- net USBGND: now reaches J42.11 (Pin_11)
- net USBGND: now also J2.11 (Pin_11)
- net AMS_AIR_M_SENS: no longer names the net of J28.7 (Pin_7)
- net AMS_AIR_PRE_SENS: no longer names the net of J28.1 (Pin_1)
- net AMS_AIR_P_SENS: no longer names the net of J28.6 (Pin_6)
- net AMS_BOOT0: no longer names the net of J42.16 (Pin_16)
- net AMS_SDC_OUT renamed SDC_AMS_IMD
- net SDC_AMS_IMD: now also J2.8 (Pin_8)
- net IMD_SDC_OUT renamed SDC_OUT
- net IR155_TSAC_GROUND renamed GND_IMD
- net GND_IMD: now also J42.23 (Pin_23)
- net SDC_TSMS_AIR renamed SDC_AIR
- net SDC_AIR: now also J2.9 (Pin_9)
- new net 24VDC_2: J33.1 (Pin_1)
- new net 24VDV_1: J2.10 (Pin_10), J42.25 (Pin_25)
- new net 24VDV_2: J42.27 (Pin_27)
- new net AIR_M_DETECTION: J2.16 (Pin_16)
- new net AIR_PRE_DETECTION: J2.15 (Pin_15)
- new net AIR_P_DETECTION: J2.14 (Pin_14)
- new net CANH_CAR: J2.5 (Pin_5), J4.2 (Pin_2), J42.36 (Pin_36)
- new net CANH_CHRG: J2.3 (Pin_3), J42.13 (Pin_13)
- new net CANL_CAR: J2.6 (Pin_6), J4.3 (Pin_3), J42.37 (Pin_37)
- new net CANL_CHRG: J2.4 (Pin_4), J42.14 (Pin_14)
- new net CAN_SH_CHRG: J42.15 (Pin_15)
- new net CHARGER_DETECTION: J2.13 (Pin_13), J42.17 (Pin_17)
- new net D+: J2.2 (Pin_2), J42.19 (Pin_19)
- new net D-: J2.1 (Pin_1), J42.18 (Pin_18)
- new net GND_2: J33.2 (Pin_2), J33.4 (Pin_4), J42.22 (Pin_22)
- new net ISABELA_+8V: J2.17 (Pin_17), J4.4 (Pin_4)
- new net ISABELA_GND: J2.7 (Pin_7), J4.1 (Pin_1)
- new net LED_IMD: J42.29 (Pin_29)
- new net SDC_IN: J2.18 (Pin_18), J42.33 (Pin_33)
- new net TSAL_GREEN: J42.20 (Pin_20), J42.21 (Pin_21)
- new net USBVDD: J2.12 (Pin_12), J42.12 (Pin_12)
- new net USB_SH: J42.28 (Pin_28)
- no-connect marks 54 -> 25
Other:
- note added: "24VDC 1"
- note added: "24VDC 2"
- note added: "AMS LED"
- note added: "CAN SHIELD CHARGER"
- note added: "CANH CHARGER"
- note added: "CANH TSAC"
- note added: "CANL CHARGER"
- note added: "CANL TSAC"
- note added: "GND 2"
- note added: "GND IMD"
- note added: "GND USB"
- note added: "GND1"
- note added: "LED IMD"
- note added: "LED TS OFF"
- note added: "SDC AIR"
- note added: "SDC IN"
- note added: "SDC OUT"
- note added: "TSAL GREEN"
- note added: "USB 5V"
- note added: "USB SHIELD"
- note removed: "24V_IN1"
- note removed: "24V_IN2"
- note removed: "600V"
- note removed: "AMS_BOOT0"
- note removed: "AMS_CANH1"
- note removed: "AMS_CANH2"
- note removed: "AMS_CANL1"
- note removed: "AMS_CANL2"
- note removed: "AMS_EXT_RESET"
- note removed: "AMS_USB_5V"
- note removed: "AMS_USB_GND"
- note removed: "CAHRGER_CANH"
- note removed: "CAHRGER_CANL"
- note removed: "GND_IN1"
- note removed: "GND_IN2"
- note removed: "IMD_DASH_LED"
- note removed: "SDC_HV_OUT"
- note removed: "SDC_RES_OUT"
- note removed: "SDC_TSMS_AIR"
- note removed: "TSAL_AIR_M_SENS"
- note removed: "TSAL_AIR_PRE_SENS"
- note removed: "TSAL_AIR_P_SENS"
- note removed: "TSAL_HV_ON"
- note removed: "x6"

Commit message: bat harness
Parts:
- removed J27, J28: Conn_01x10, symbol Connector_Generic:Conn_01x10
- removed J29, J30, J31: CABLE, symbol Connector:Conn_01x04_Pin
- removed J3: M80-5100642, symbol Connector_Generic:Conn_01x08
- added J5, J6: Conn_01x06, symbol Connector_Generic:Conn_01x06
Connections:
- net LED_IMD is gone; now on net IMD_LED: J42.29 (Pin_29)
- net GND_1: now also J2.19 (Pin_19)
- net IMD_DASH_LED renamed IMD_LED
- new net AIR_M+: J5.4 (Pin_4)
- new net AIR_M-: J5.1 (Pin_1)
- new net AIR_P+: J5.5 (Pin_5)
- new net AIR_P-: J5.2 (Pin_2)
- new net AIR_PRE+: J5.6 (Pin_6)
- new net AIR_PRE-: J5.3 (Pin_3)
- no-connect marks 25 -> 24
